File: hardware/_autosave-boombox.kicad_sch (KiCad schematic)
At the start: 36 parts, among them J1 Micro_SD_Card_Det1, J4 USB_C_Receptacle_USB2.0_16P, SW1 SW_SPST, SW2 SW_SPST, SW3 SW_SPST, SW4 SW_SPST, SW5 SW_SPST, U1 Pico, U2 TMAG5231, U3 TMAG5231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

Commit message: values
Other:
- title: (none) -> Boombuddy
Changed lines of the file:
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@@
 	(generator_version "8.0")
 	(paper "A4")
+	(title_block
+		(title "Boombuddy")
+	)
 	(junction
 		(at 105.41 146.05)
