File: hardware/_autosave-boombox.kicad_pcb (KiCad board)
At the start: 4 copper layers, 95 x 70 mm, 76 parts, among them J1 Micro_SD_Card_Det1, J2 AudioJack4, J3 Battery, J4 USB_C_Receptacle_USB2.0_16P, SW1 SW_SPST, SW2 SW_SPST, SW3 SW_SPST, SW4 SW_SPST, SW5 SW_SPST, U1 Pico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

Commit message: .
Parts:
- removed R12, R5: 100k, Resistor_SMD:R_0402_1005Metric_Pad0.72x0.64mm_HandSolder
- J2: renamed from LS1; value Speaker -> AudioJack4; footprint boombox:EBAA02C -> boombox:EBAA02C_Audio
- LS1: renamed from J2; value AudioJack4 -> Speaker; footprint boombox:EBAA02C_Audio -> boombox:EBAA02C
- R13, R14, R15, R16: moved to B.Cu
- moved C23 83.2 mm to (174.3, 82.7), turned to 180 degrees
- moved R13 80.9 mm to (155.8, 105.0), turned to 90 degrees
- moved R14 75.5 mm to (158.3, 105.2), turned to 90 degrees
- moved C19 75.3 mm to (174.6, 84.0), turned to 180 degrees
- moved R15 67.7 mm to (163.3, 105.0), turned to 90 degrees
- moved C22 65.3 mm to (185.5, 85.1), turned to -90 degrees
- moved R16 65.2 mm to (168.2, 80.5), turned to 0 degrees
- moved C18 63.6 mm to (184.0, 85.0), turned to -90 degrees
- moved U8 53.6 mm to (177.6, 82.3)
- moved U10 52.2 mm to (182.5, 82.3)
- moved SW2 25.4 mm to (133.9, 55.8)
- moved SW3 25.3 mm to (147.0, 55.8)
- moved SW1 22.8 mm to (100.3, 37.0)
- moved Q3 18.9 mm to (163.2, 80.6)
- moved C6 4.51 mm to (159.9, 45.8)
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Connections:
- SW2 pad 2: unconnected-(SW2-B-Pad2)_1 -> SLP_PWR
- SW3 pad 2: unconnected-(SW3-B-Pad2)_1 -> SLP_PWR
- SW4 pad 2: unconnected-(SW4-B-Pad2) -> SLP_PWR
- SW5 pad 2: unconnected-(SW5-B-Pad2) -> SLP_PWR
- U10 pad B3: Net-(U10-GAIN_SLOT) -> VCC
- U8 pad B3: Net-(U8-GAIN_SLOT) -> VCC
Routing:
- net Net-(U1-GPIO5): track 62.3 -> 2.98 mm
- net Net-(U1-GPIO4): track 59.1 -> 3.73 mm
- net Net-(U10-DAI1): track 2.35 -> 49.9 mm, vias 0 -> 5
- net Net-(U10-DAI0): track 5.57 -> 51.8 mm, vias 0 -> 4
- net /Power/MAG_SENSOR2: track 57.2 -> 12.4 mm
- net Net-(U10-DAI2): track 3.30 -> 46.9 mm, vias 0 -> 5
- net /Audio/HEADPHONE_EN: track 0.00 -> 35.7 mm, vias 0 -> 2
- net VCC: track 213.9 -> 246.4 mm, vias 6 -> 7
- net /Power/MAG_SENSOR1: track 42.6 -> 17.1 mm, vias 2 -> 1
- net /Audio/~{HEADPHONE_DETECT}: track 22.3 -> 44.5 mm, vias 0 -> 2
- net /Power/CLOCK_ALARM: track 81.6 -> 60.5 mm, vias 4 -> 2
- net /Audio/SPEAKER_EN: track 0.00 -> 18.8 mm
- net SLP_PWR: track 257.4 -> 239.5 mm, vias 11 -> 12
- net Net-(U10-OUTN): track 0.00 -> 11.2 mm
- net Net-(U10-OUTP): track 0.00 -> 9.25 mm
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Other:
- board size 95 x 70 mm -> 97.7 x 88.3 mm
