File: hardware/audio.kicad_sch (KiCad schematic)
At the start: 16 parts, among them J2 AudioJack4, U10 MAX98365A, U8 MAX98365A

Commit message: Comitting so Nate can see errors
Parts:
- U10, U8: footprint (none) -> boombox:MAX98365

Commit message: Routing
Parts:
- J2: footprint boombox:Degson 3 Pin -> boombox:EBAA02C_Audio; symbol Connector_Audio:AudioJack4 -> Connector_Audio:AudioJack2
- LS1: footprint boombox:Degson 3 Pin -> boombox:EBAA02C
Connections:
- no-connect marks 2 -> 0
Changed lines of the file:
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@@
 	)
 	(junction
-		(at 168.91 55.88)
+		(at 168.91 58.42)
 		(diameter 0)
 		(color 0 0 0 0)
 	)
-	(no_connect
-		(at 175.26 60.96)
-	)
-	(no_connect
-		(at 175.26 58.42)
-	)
 	(wire
 		(pts
@@
 	(wire
 		(pts
-			(xy 161.29 63.5) (xy 175.26 63.5)
+			(xy 161.29 60.96) (xy 175.26 60.96)
 		)
 		(stroke
@@
 	(wire
 		(pts
-			(xy 168.91 40.64) (xy 168.91 55.88)
+			(xy 168.91 40.64) (xy 168.91 58.42)
 		)
 		(stroke
@@
 	(wire
 		(pts
-			(xy 161.29 63.5) (xy 161.29 60.96)
-		)
-		(stroke
-			(width 0)
-			(type default)
-		)
-	)
-	(wire
-		(pts
 			(xy 186.69 137.16) (xy 189.23 137.16)
 		)
@@
 	(wire
 		(pts
-			(xy 161.29 55.88) (xy 161.29 58.42)
-		)
-		(stroke
-			(width 0)
-			(type default)
-		)
-	)
-	(wire
-		(pts
 			(xy 121.92 125.73) (xy 130.81 125.73)
 		)
@@
 	(wire
 		(pts
-			(xy 161.29 55.88) (xy 168.91 55.88)
+			(xy 161.29 58.42) (xy 168.91 58.42)
 		)
 		(stroke
@@
 	(wire
 		(pts
-			(xy 168.91 55.88) (xy 175.26 55.88)
+			(xy 168.91 58.42) (xy 175.26 58.42)
 		)
 		(stroke
@@
 			)
 		)
-		(property "Footprint" "boombox:Degson 3 Pin"
+		(property "Footprint" "boombox:EBAA02C"
 			(at 214.63 119.38 0)
 			(effects
@@
 	)
 	(symbol
-		(lib_id "Connector_Audio:AudioJack4")
-		(at 180.34 60.96 180)
+		(lib_id "Connector_Audio:AudioJack2")
+		(at 180.34 58.42 180)
 		(unit 1)
 		(exclude_from_sim no)
@@
 		(dnp no)
 		(property "Reference" "J2"
-			(at 182.88 69.85 0)
+			(at 182.88 67.31 0)
 			(effects
 				(font
@@
 		)
 		(property "Value" "AudioJack4"
-			(at 182.88 67.31 0)
-			(effects
-				(font
-					(size 1.27 1.27)
-				)
-			)
-		)
-		(property "Footprint" "boombox:Degson 3 Pin"
-			(at 180.34 60.96 0)
-			(effects
-				(font
-					(size 1.27 1.27)
-				)
-				(hide yes)
-			)
-		)
-		(property "Datasheet" "${KIPRJMOD}/datasheets/headphone.pdf"
-			(at 180.34 60.96 0)
-			(effects
-				(font
-					(size 1.27 1.27)
-				)
-				(hide yes)
-			)
-		)
-		(property "Description" "Audio Jack, 4 Poles (TRRS)"
-			(at 180.34 60.96 0)
+			(at 182.88 64.77 0)
+			(effects
+				(font
+					(size 1.27 1.27)
+				)
+			)
+		)
+		(property "Footprint" "boombox:EBAA02C_Audio"
+			(at 180.34 58.42 0)
+			(effects
+				(font
+					(size 1.27 1.27)
+				)
+				(hide yes)
+			)
+		)
+		(property "Datasheet" "~"
+			(at 180.34 58.42 0)
+			(effects
+				(font
+					(size 1.27 1.27)
+				)
+				(hide yes)
+			)
+		)
+		(property "Description" "Audio Jack, 2 Poles (Mono / TS)"
+			(at 180.34 58.42 0)
 			(effects
 				(font
@@
 		)
 		(property "Sim.Device" ""
-			(at 180.34 60.96 0)
+			(at 180.34 58.42 0)
 			(effects
 				(font
@@
 		)
 		(property "Sim.Pins" ""
-			(at 180.34 60.96 0)
+			(at 180.34 58.42 0)
 			(effects
 				(font
@@
 		(pin "S"
 		)
-		(pin "R2"
-		)
-		(pin "R1"
-		)
-		(instances
+		(instances

Commit message: .
Parts:
- removed R12, R5: 100k, Resistor_SMD:R_0402_1005Metric_Pad0.72x0.64mm_HandSolder, symbol Device:R_US
- removed R15: 0, Resistor_SMD:R_0402_1005Metric_Pad0.72x0.64mm_HandSolder, symbol Device:R_US
Connections:
- net VCC: now also U10.B3 (GAIN_SLOT), U8.B3 (GAIN_SLOT)
- net ~{HEADPHONE_DETECT}: now also J2.S; no longer J2.T
- net at U8.A2 (OUTN): now also J2.T; no longer J2.S
Other:
- moved on the sheet: J2

Commit message: Switches
Parts:
- added R12: 0, Resistor_SMD:R_0402_1005Metric_Pad0.72x0.64mm_HandSolder, symbol Device:R_US
Connections:
- net I2S_BCLK: now also R12.1
- net at U10.A4 (DAI2), U8.A4 (DAI2): now also R12.2
Changed lines of the file:
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@@
+	)
+	(symbol
+		(lib_id "Device:R_US")
+		(at 118.11 125.73 90)
+		(unit 1)
+		(exclude_from_sim no)
+		(in_bom yes)
+		(on_board yes)
+		(dnp no)
+		(fields_autoplaced yes)
+		(property "Reference" "R12"
+			(at 118.11 119.38 90)
+			(effects
+				(font
+					(size 1.27 1.27)
+				)
+			)
+		)
+		(property "Value" "0"
+			(at 118.11 121.92 90)
+			(effects
+				(font
+					(size 1.27 1.27)
+				)
+			)
+		)
+		(property "Footprint" "Resistor_SMD:R_0402_1005Metric_Pad0.72x0.64mm_HandSolder"
+			(at 118.364 124.714 90)
+			(effects
+				(font
+					(size 1.27 1.27)
+				)
+				(hide yes)
+			)
+		)
+		(property "Datasheet" "~"
+			(at 118.11 125.73 0)
+			(effects
+				(font
+					(size 1.27 1.27)
+				)
+				(hide yes)
+			)
+		)
+		(property "Description" "Resistor, US symbol"
+			(at 118.11 125.73 0)
+			(effects
+				(font
+					(size 1.27 1.27)
+				)
+				(hide yes)
+			)
+		)
+		(property "Sim.Device" ""
+			(at 118.11 125.73 0)
+			(effects
+				(font
+					(size 1.27 1.27)
+				)
+				(hide yes)
+			)
+		)
+		(property "Sim.Pins" ""
+			(at 118.11 125.73 0)
+			(effects
+				(font
+					(size 1.27 1.27)
+				)
+				(hide yes)
+			)
+		)
+		(pin "2"
+		)
+		(pin "1"
+		)
+		(instances
+			(project "boombox"
+				(path "/947839cd-c3fd-4edc-874b-58f50b880ae8/1df97fe1-ae1c-48c8-898d-06b71dd703d8"
+					(reference "R12")
+					(unit 1)
+				)
+			)
+		)
 	)
 	(symbol
