File: hardware/boombox.kicad_pcb (KiCad board)
At the start: 4 copper layers, 125 x 107.3 mm, 86 parts, among them J1 Micro_SD_Card_Det1, J2 Screw_Terminal_01x07, J4 USB_C_Receptacle_USB2.0_16P, J5 Screw_Terminal_01x07, U1 Pico, U10 MAX98365A, U2 TMAG5231, U3 TMAG5231, U4 TMAG5231, U5 TMAG5231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

Commit message: .
Connections:
- Q6 pad 2: /Power/CLOCK_ALARM -> GND
- Q6 pad 3: GND -> /Power/CLOCK_ALARM
Routing:
- net /Power/CLOCK_ALARM: track 95.6 -> 91.5 mm, vias 2 -> 3
- net /Power/~{POWER_OFF}: track 68.0 -> 66.2 mm
- net GND: track 100.9 -> 99.2 mm, vias 36 -> 35
Changed lines of the file:
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@@
 	(net 79 "unconnected-(S5-NO_2-Pad6)")
 	(net 80 "Net-(S1-NC_1)")
+	(net 81 "unconnected-(U1-ADC_VREF-Pad35)")
+	(net 82 "unconnected-(U1-VBUS-Pad40)")
+	(net 83 "unconnected-(U1-RUN-Pad30)_1")
+	(net 84 "unconnected-(U1-3V3_EN-Pad37)_1")
 	(footprint "Resistor_SMD:R_0402_1005Metric_Pad0.72x0.64mm_HandSolder"
 		(layer "F.Cu")
@@
 			(layers "F.Cu" "F.Paste" "F.Mask")
 			(roundrect_rratio 0.25)
-			(net 32 "/Power/CLOCK_ALARM")
+			(net 1 "GND")
 			(pinfunction "S")
 			(pintype "passive")
@@
 			(layers "F.Cu" "F.Paste" "F.Mask")
 			(roundrect_rratio 0.25)
-			(net 1 "GND")
+			(net 32 "/Power/CLOCK_ALARM")
 			(pinfunction "D")
 			(pintype "passive")
@@
 			(layers "*.Cu" "*.Mask")
 			(remove_unused_layers no)
-			(net 48 "unconnected-(U1-RUN-Pad30)")
+			(net 83 "unconnected-(U1-RUN-Pad30)_1")
 			(pinfunction "RUN")
 			(pintype "input+no_connect")
@@
 			(layers "*.Cu" "*.Mask")
 			(remove_unused_layers no)
-			(net 46 "unconnected-(U1-ADC_VREF-Pad35)_1")
+			(net 81 "unconnected-(U1-ADC_VREF-Pad35)")
 			(pinfunction "ADC_VREF")
 			(pintype "power_in+no_connect")
@@
 			)
 			(layers "F.Cu" "F.Mask")
-			(net 44 "unconnected-(U1-3V3_EN-Pad37)")
+			(net 84 "unconnected-(U1-3V3_EN-Pad37)_1")
 			(pinfunction "3V3_EN")
 			(pintype "input+no_connect")
@@
 			)
 			(layers "F.Cu" "F.Mask")
-			(net 49 "unconnected-(U1-VBUS-Pad40)_1")
+			(net 82 "unconnected-(U1-VBUS-Pad40)")
 			(pinfunction "VBUS")
 			(pintype "power_in+no_connect")
@@
 	)
 	(segment
+		(start 131.8 92.85)
+		(end 131.75 92.8)
+		(width 0.6)
+		(layer "F.Cu")
+		(net 1)
+	)
+	(segment
 		(start 177.38375 82.1175)
 		(end 177.38375 82.5175)
@@
 		(net 1)
 	)
-	(segment
-		(start 133.625 91.85)
-		(end 135.475 91.85)
-		(width 0.6)
-		(layer "F.Cu")
-		(net 1)
-	)
 	(via
 		(at 165.475 131.825)
@@
 	)
 	(via
-		(at 135.475 91.85)
-		(size 1)
-		(drill 0.6)
-		(layers "F.Cu" "B.Cu")
-		(net 1)
-	)
-	(via
 		(at 167.9 131.825)
 		(size 0.45)
@@
 	)
 	(segment
-		(start 129.925 90.9)
-		(end 131.75 90.9)
-		(width 0.6)
-		(layer "F.Cu")
-		(net 2)
-	)
-	(segment
 		(start 129.925 89.55)
 		(end 129.925 90.9)
@@
 	)
 	(segment
-		(start 131.8 92.85)
-		(end 131.75 92.8)
-		(width 0.6)
-		(layer "F.Cu")
-		(net 32)
-	)
-	(segment
 		(start 142.454407 81.5)
 		(end 138.8994 81.5)
@@
 	)
 	(segment
-		(start 135.889214 92.85)
-		(end 131.8 92.85)
-		(width 0.6)
-		(layer "F.Cu")
-		(net 32)
-	)
-	(segment
 		(start 164.1375 81.5125)
 		(end 142.466907 81.5125)
@@
 	)
 	(segment
-		(start 129.925 92.8)
-		(end 131.75 92.8)
-		(width 0.6)
-		(layer "F.Cu")
-		(net 32)
-	)
-	(segment
 		(start 142.466907 81.5125)
 		(end 142.454407 81.5)
@@
 	)
 	(segment
+		(start 133.625 91.85)
+		(end 135.475 91.85)
+		(width 0.6)
+		(layer "F.Cu")
+		(net 32)
+	)
+	(segment
 		(start 136.475 91.137501)
 		(end 136.475 92.264214)
@@
 		(size 1)
 		(drill 0.6)
+		(layers "F.Cu" "B.Cu")
+		(net 32)
+	)
+	(via
+		(at 135.475 91.85)
+		(size 1)
+		(drill 0.6)
