File: hardware/boombox.kicad_sch (KiCad schematic)
At the start: 44 parts, among them J1 Micro_SD_Card_Det1, J2 Screw_Terminal_01x07, J4 USB_C_Receptacle_USB2.0_16P, U1 Pico, U2 TMAG5231, U3 TMAG5231, U4 TMAG5231, U5 TMAG5231, U6 TMAG5231, U7 MCP7940MT-I/SN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

Commit message: .
Connections:
- net at R7.2, U7.6 (SCL): now also U1.7 (GPIO5); no longer U1.6 (GPIO4)
- net at R6.2, U7.5 (SDA): now also U1.6 (GPIO4); no longer U1.7 (GPIO5)
Changed lines of the file:
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@@
+	)
+	(junction
+		(at 91.44 33.02)
+		(diameter 0)
+		(color 0 0 0 0)
 	)
 	(junction
@@
 	)
 	(junction
-		(at 91.44 33.02)
-		(diameter 0)
-		(color 0 0 0 0)
-	)
-	(junction
 		(at 124.46 132.08)
 		(diameter 0)
@@
 	(wire
 		(pts
+			(xy 91.44 33.02) (xy 91.44 86.36)
+		)
+		(stroke
+			(width 0)
+			(type default)
+		)
+	)
+	(wire
+		(pts
 			(xy 82.55 52.07) (xy 93.98 52.07)
 		)
@@
 	(wire
 		(pts
-			(xy 88.9 86.36) (xy 88.9 35.56)
-		)
-		(stroke
-			(width 0)
-			(type default)
-		)
-	)
-	(wire
-		(pts
 			(xy 194.31 91.44) (xy 173.99 91.44)
 		)
@@
 	(wire
 		(pts
+			(xy 91.44 86.36) (xy 138.43 86.36)
+		)
+		(stroke
+			(width 0)
+			(type default)
+		)
+	)
+	(wire
+		(pts
 			(xy 78.74 166.37) (xy 78.74 168.91)
 		)
@@
 	(wire
 		(pts
-			(xy 88.9 86.36) (xy 138.43 86.36)
-		)
-		(stroke
-			(width 0)
-			(type default)
-		)
-	)
-	(wire
-		(pts
 			(xy 120.65 45.72) (xy 121.92 45.72)
 		)
@@
 	(wire
 		(pts
-			(xy 91.44 33.02) (xy 91.44 83.82)
-		)
-		(stroke
-			(width 0)
-			(type default)
-		)
-	)
-	(wire
-		(pts
 			(xy 33.02 27.94) (xy 46.99 27.94)
 		)
@@
 	(wire
 		(pts
+			(xy 88.9 83.82) (xy 138.43 83.82)
+		)
+		(stroke
+			(width 0)
+			(type default)
+		)
+	)
+	(wire
+		(pts
+			(xy 88.9 35.56) (xy 88.9 83.82)
+		)
+		(stroke
+			(width 0)
+			(type default)
+		)
+	)
+	(wire
+		(pts
 			(xy 66.04 97.79) (xy 66.04 124.46)
 		)
@@
 		)
 	)
-	(wire
-		(pts
-			(xy 91.44 83.82) (xy 138.43 83.82)
-		)
-		(stroke
-			(width 0)
-			(type default)
-		)
-	)
