File: hardware/boombox.kicad_sch (KiCad schematic)
At the start: 44 parts, among them J1 Micro_SD_Card_Det1, J2 Screw_Terminal_01x07, J4 USB_C_Receptacle_USB2.0_16P, U1 Pico, U2 TMAG5231, U3 TMAG5231, U4 TMAG5231, U5 TMAG5231, U6 TMAG5231, U7 MCP7940MT-I/SN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

Commit message: speaker
Parts:
- R6, R7: value 10k -> 5.1k
Connections:
- net Audio/I2S_BCLK: now also U1.27 (GPIO21); no longer U1.29 (GPIO22)
- net Audio/I2S_DOUT: now also U1.26 (GPIO20); no longer U1.27 (GPIO21)
- net Audio/I2S_LRCLK: now also U1.29 (GPIO22); no longer U1.26 (GPIO20)
Changed lines of the file:
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@@
 	(wire
 		(pts
-			(xy 196.85 99.06) (xy 173.99 99.06)
-		)
-		(stroke
-			(width 0)
-			(type default)
-		)
-	)
-	(wire
-		(pts
 			(xy 209.55 109.22) (xy 173.99 109.22)
 		)
@@
 	(wire
 		(pts
-			(xy 194.31 91.44) (xy 173.99 91.44)
-		)
-		(stroke
-			(width 0)
-			(type default)
-		)
-	)
-	(wire
-		(pts
 			(xy 69.85 99.06) (xy 138.43 99.06)
 		)
@@
 	(wire
 		(pts
-			(xy 91.44 86.36) (xy 138.43 86.36)
+			(xy 199.39 104.14) (xy 173.99 104.14)
 		)
 		(stroke
@@
 	(wire
 		(pts
-			(xy 78.74 166.37) (xy 78.74 168.91)
+			(xy 201.93 74.93) (xy 201.93 106.68)
 		)
 		(stroke
@@
 	(wire
 		(pts
-			(xy 201.93 74.93) (xy 201.93 106.68)
+			(xy 196.85 69.85) (xy 196.85 99.06)
+		)
+		(stroke
+			(width 0)
+			(type default)
+		)
+	)
+	(wire
+		(pts
+			(xy 91.44 86.36) (xy 138.43 86.36)
+		)
+		(stroke
+			(width 0)
+			(type default)
+		)
+	)
+	(wire
+		(pts
+			(xy 78.74 166.37) (xy 78.74 168.91)
 		)
 		(stroke
@@
 	(wire
 		(pts
-			(xy 176.53 88.9) (xy 176.53 101.6)
+			(xy 196.85 99.06) (xy 173.99 99.06)
 		)
 		(stroke
@@
 	(wire
 		(pts
-			(xy 52.07 88.9) (xy 20.32 88.9)
+			(xy 176.53 88.9) (xy 176.53 101.6)
 		)
 		(stroke
@@
 	(wire
 		(pts
-			(xy 99.06 88.9) (xy 138.43 88.9)
+			(xy 52.07 88.9) (xy 20.32 88.9)
 		)
 		(stroke
@@
 		)
 	)
-	(bus
+	(wire
 		(pts
-			(xy 48.26 74.93) (xy 55.88 74.93)
+			(xy 99.06 88.9) (xy 138.43 88.9)
 		)
 		(stroke
@@
 		)
 	)
-	(wire
+	(bus
 		(pts
-			(xy 204.47 120.65) (xy 204.47 93.98)
+			(xy 48.26 74.93) (xy 55.88 74.93)
 		)
 		(stroke
@@
 	(wire
 		(pts
-			(xy 199.39 104.14) (xy 173.99 104.14)
+			(xy 194.31 120.65) (xy 194.31 93.98)
 		)
 		(stroke
@@
 	(wire
 		(pts
-			(xy 196.85 69.85) (xy 196.85 99.06)
+			(xy 199.39 72.39) (xy 199.39 104.14)
 		)
 		(stroke
@@
 	(wire
 		(pts
-			(xy 204.47 93.98) (xy 173.99 93.98)
+			(xy 194.31 93.98) (xy 173.99 93.98)
 		)
 		(stroke
@@
 	(wire
 		(pts
+			(xy 173.99 91.44) (xy 194.31 91.44)
+		)
+		(stroke
+			(width 0)
+			(type default)
+		)
+	)
+	(wire
+		(pts
 			(xy 102.87 58.42) (xy 105.41 58.42)
 		)
@@
 	(wire
 		(pts
-			(xy 251.46 72.39) (xy 199.39 72.39)
+			(xy 251.46 74.93) (xy 201.93 74.93)
 		)
 		(stroke
@@
 	(wire
 		(pts
-			(xy 251.46 69.85) (xy 196.85 69.85)
+			(xy 251.46 72.39) (xy 199.39 72.39)
 		)
 		(stroke
@@
 	(wire
 		(pts
-			(xy 199.39 72.39) (xy 199.39 104.14)
-		)
-		(stroke
-			(width 0)
-			(type default)
-		)
-	)
-	(wire
-		(pts
 			(xy 48.26 64.77) (xy 71.12 64.77)
 		)
@@
 	(wire
 		(pts
-			(xy 251.46 74.93) (xy 201.93 74.93)
+			(xy 251.46 69.85) (xy 196.85 69.85)
 		)
 		(stroke
@@
 	(wire
 		(pts
+			(xy 201.93 106.68) (xy 173.99 106.68)
+		)
+		(stroke
+			(width 0)
+			(type default)
+		)
+	)
+	(wire
+		(pts
 			(xy 66.04 97.79) (xy 66.04 124.46)
 		)
@@
 	(wire
 		(pts
-			(xy 201.93 106.68) (xy 173.99 106.68)
-		)
-		(stroke
-			(width 0)
-			(type default)
-		)
-	)
-	(wire
-		(pts
 			(xy 58.42 95.25) (xy 58.42 99.06)
 		)
@@
 	(wire
 		(pts
-			(xy 214.63 120.65) (xy 204.47 120.65)
+			(xy 214.63 120.65) (xy 194.31 120.65)
 		)
 		(stroke
@@
 			)
 		)
-		(property "Value" "10k"
+		(property "Value" "5.1k"
 			(at 93.98 26.6699 0)
 			(effects
@@
 			)
 		)
-		(property "Value" "10k"
+		(property "Value" "5.1k"
 			(at 85.09 26.6699 0)
 			(effects
@@
 		)
 		(pin "I2S_BCLK" input
-			(at 251.46 69.85 180)
+			(at 251.46 72.39 180)
 			(effects
 				(font
@@
 		)
 		(pin "I2S_DOUT" input
-			(at 251.46 72.39 180)
+			(at 251.46 74.93 180)
 			(effects
 				(font
@@
 		)
 		(pin "I2S_LRCLK" input
-			(at 251.46 74.93 180)
+			(at 251.46 69.85 180)
 			(effects
 				(font
