File: hardware/power.kicad_sch (KiCad schematic)
At the start: 23 parts, among them U9 MCP73811T-420I-OT

Commit message: Flipped mosfet
Connections:
- net CLOCK_ALARM: now also Q6.3 (D); no longer Q6.2 (S)
- net GND: now also Q6.2 (S); no longer Q6.3 (D)
Other:
- moved on the sheet: Q6
Changed lines of the file:
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@@
 	(symbol
 		(lib_id "boombox:DMN2310U-7")
-		(at 193.04 74.93 180)
+		(at 193.04 74.93 0)
+		(mirror y)
 		(unit 1)
 		(exclude_from_sim no)
@@
 		(on_board yes)
 		(dnp no)
-		(fields_autoplaced yes)
 		(property "Reference" "Q6"
-			(at 187.96 74.2949 0)
+			(at 187.96 75.5651 0)
 			(effects
 				(font
@@
 		)
 		(property "Value" "~"
-			(at 187.96 76.2 0)
+			(at 187.96 73.66 0)
 			(effects
 				(font
@@
 		)
 		(property "Footprint" "Package_TO_SOT_SMD:SOT-23"
-			(at 191.77 60.452 0)
+			(at 191.77 89.408 0)
 			(effects
 				(font

Commit message: speaker
Parts:
- added Q8: ~, Package_TO_SOT_SMD:SOT-23, symbol boombox:DMN2310U-7
- added R15: 1M, Resistor_SMD:R_0402_1005Metric_Pad0.72x0.64mm_HandSolder, symbol Device:R_US
- C1: value 6pF -> 0.1uF
- C2: value 1nF -> 0.1uF
- D11: now not fitted
Connections:
- net GND: now also Q8.2 (S), R15.2
- net ~{POWER_OFF}: now also Q8.1 (G), R15.1; no longer C1.1, Q4.3 (D), Q6.1 (G), R1.2
- new net: C1.1, Q4.3 (D), Q6.1 (G), Q8.3 (D), R1.2
